Commit message: rotate ur_connector

File: cob_description/urdf/ur_connector/ur_connector.urdf.xacro (robot description, xacro)
@@ -35,5 +35,5 @@
 		<!-- joint between base_link and ur_connector_link -->
 		<joint name="${name}_joint" type="revolute">
-			<origin xyz="-0.0201 -0.1736 0.136" rpy="0 0 0"/>
+			<origin xyz="-0.0201 -0.1736 0.136" rpy="0 0 2.7926"/>
 			<parent link="${name}_fixed_link"/>
 			<child link="${name}_link"/>
